Commit message: Add more performant model

File: bobnet_descriptions/spot_description/urdf/spot.urdf (robot description, URDF)
Before this commit: robot spot, 18 links, 17 joints
Links:
- link LF_FOOT: mass None -> 0.215; geometry collision sphere radius=0.035
- link LH_FOOT: mass None -> 0.215; geometry collision sphere radius=0.035
- link RF_FOOT: mass None -> 0.215; geometry collision sphere radius=0.035
- link RH_FOOT: mass None -> 0.215; geometry collision sphere radius=0.035
- link fl_lleg: geometry collision cylinder length=0.30 radius=0.03; visual mesh filename=package://spot_description/meshes/visual/fl_lleg.dae
- link fl_uleg: geometry collision cylinder length=0.3 radius=0.05; visual mesh filename=package://spot_description/meshes/visual/fl_uleg.dae
- link fr_lleg: geometry collision cylinder length=0.30 radius=0.03; visual mesh filename=package://spot_description/meshes/visual/fr_lleg.dae
- link fr_uleg: geometry collision cylinder length=0.3 radius=0.05; visual mesh filename=package://spot_description/meshes/visual/fr_uleg.dae
- link hl_lleg: geometry collision cylinder length=0.30 radius=0.03; visual mesh filename=package://spot_description/meshes/visual/hl_lleg.dae
- link hl_uleg: geometry collision cylinder length=0.3 radius=0.05; visual mesh filename=package://spot_description/meshes/visual/hl_uleg.dae
- link hr_lleg: geometry collision cylinder length=0.30 radius=0.03; visual mesh filename=package://spot_description/meshes/visual/hr_lleg.dae
- link hr_uleg: geometry collision cylinder length=0.3 radius=0.05; visual mesh filename=package://spot_description/meshes/visual/hr_uleg.dae
Joints:
- joint LF_HAA: limit lower=-0.78539816339744827899 upper=0.78539816339744827899 effort=80 velocity=7.5 -> lower=-10.78539816339744827899 upper=10.78539816339744827899 effort=100 velocity=7.5
- joint LF_HFE: limit lower=-0.89884456477707963539 upper=2.2951079663725435509 effort=80 velocity=7.5 -> lower=-10.89884456477707963539 upper=12.2951079663725435509 effort=100 velocity=7.5
- joint LF_KFE: limit lower=-2.7929 upper=-0.254402 effort=80 velocity=7.5 -> lower=-12.7929 upper=12.7929 effort=100 velocity=7.5
- joint LH_HAA: limit lower=-0.78539816339744827899 upper=0.78539816339744827899 effort=80 velocity=7.5 -> lower=-10.78539816339744827899 upper=10.78539816339744827899 effort=100 velocity=7.5
- joint LH_HFE: limit lower=-0.89884456477707963539 upper=2.2951079663725435509 effort=80 velocity=7.5 -> lower=-10.89884456477707963539 upper=12.2951079663725435509 effort=100 velocity=7.5
- joint LH_KFE: limit lower=-2.7929 upper=-0.254402 effort=80 velocity=7.5 -> lower=-12.7929 upper=12.7929 effort=100 velocity=7.5
- joint RF_HAA: limit lower=-0.78539816339744827899 upper=0.78539816339744827899 effort=80 velocity=7.5 -> lower=-10.78539816339744827899 upper=10.78539816339744827899 effort=100 velocity=7.5
- joint RF_HFE: limit lower=-0.89884456477707963539 upper=2.2951079663725435509 effort=80 velocity=7.5 -> lower=-10.898845 upper=12.24363 effort=100 velocity=7.5
- joint RF_KFE: limit lower=-2.7929 upper=-0.254402 effort=80 velocity=7.5 -> lower=-12.7929 upper=12.7929 effort=100 velocity=7.5
- joint RH_HAA: limit lower=-0.78539816339744827899 upper=0.78539816339744827899 effort=80 velocity=7.5 -> lower=-10.78539816339744827899 upper=10.78539816339744827899 effort=100 velocity=7.5
- joint RH_HFE: limit lower=-0.89884456477707963539 upper=2.2951079663725435509 effort=80 velocity=7.5 -> lower=-10.89884456477707963539 upper=12.2951079663725435509 effort=100 velocity=7.5
- joint RH_KFE: limit lower=-2.7929 upper=-0.254402 effort=80 velocity=7.5 -> lower=-12.7929 upper=12.7929 effort=100 velocity=7.5

Commit message: Update urdfs

File: bobnet_descriptions/spot_description/urdf/spot.urdf (robot description, URDF)
Before this commit: robot spot, 18 links, 17 joints
Joints:
- joint LF_HAA: limit lower=-10.78539816339744827899 upper=10.78539816339744827899 effort=100 velocity=7.5 -> lower=-0.78539816339744827899 upper=0.78539816339744827899 effort=80 velocity=7.5
- joint LF_HFE: limit lower=-10.89884456477707963539 upper=12.2951079663725435509 effort=100 velocity=7.5 -> lower=-0.89884456477707963539 upper=2.2951079663725435509 effort=80 velocity=7.5
- joint LF_KFE: limit lower=-12.7929 upper=12.7929 effort=100 velocity=7.5 -> lower=-2.7929 upper=-0.267153 effort=80 velocity=7.5
- joint LH_HAA: limit lower=-10.78539816339744827899 upper=10.78539816339744827899 effort=100 velocity=7.5 -> lower=-0.78539816339744827899 upper=0.78539816339744827899 effort=80 velocity=7.5
- joint LH_HFE: limit lower=-10.89884456477707963539 upper=12.2951079663725435509 effort=100 velocity=7.5 -> lower=-0.89884456477707963539 upper=2.2951079663725435509 effort=80 velocity=7.5
- joint LH_KFE: limit lower=-12.7929 upper=12.7929 effort=100 velocity=7.5 -> lower=-2.7929 upper=-0.267153 effort=80 velocity=7.5
- joint RF_HAA: limit lower=-10.78539816339744827899 upper=10.78539816339744827899 effort=100 velocity=7.5 -> lower=-0.78539816339744827899 upper=0.78539816339744827899 effort=80 velocity=7.5
- joint RF_HFE: limit lower=-10.898845 upper=12.24363 effort=100 velocity=7.5 -> lower=-0.89884456477707963539 upper=2.2951079663725435509 effort=80 velocity=7.5
- joint RF_KFE: limit lower=-12.7929 upper=12.7929 effort=100 velocity=7.5 -> lower=-2.7929 upper=-0.267153 effort=80 velocity=7.5
- joint RH_HAA: limit lower=-10.78539816339744827899 upper=10.78539816339744827899 effort=100 velocity=7.5 -> lower=-0.78539816339744827899 upper=0.78539816339744827899 effort=80 velocity=7.5
- joint RH_HFE: limit lower=-10.89884456477707963539 upper=12.2951079663725435509 effort=100 velocity=7.5 -> lower=-0.89884456477707963539 upper=2.2951079663725435509 effort=80 velocity=7.5
- joint RH_KFE: limit lower=-12.7929 upper=12.7929 effort=100 velocity=7.5 -> lower=-2.7929 upper=-0.267153 effort=80 velocity=7.5
